File: electrical/pfd.kicad_sch (KiCad schematic)
At the start: 9 parts

Commit message: Added lighting bus
Connections:
- net LIGHTS_HI: now reaches GDU460.P4X02_43 (14V_LIGHTING_BUS_HI)
Changed lines of the file:
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@@
 	(title_block
 		(title "PFD & ADAHRS")
-		(date "2025-10-12")
-		(rev "1.1.8")
+		(date "2025-10-19")
+		(rev "1.1.15")
 		(company "N78HR")
 	)
@@
 		(pts
 			(xy 120.65 127) (xy 144.78 127)
+		)
+		(stroke
+			(width 0)
+			(type default)
+		)
+	)
+	(wire
+		(pts
+			(xy 62.23 80.01) (xy 68.58 80.01)
 		)
 		(stroke
@@
 		(effects
 			(font
+				(size 1.27 1.27)
+			)
+			(justify left)
+		)
+	)
+	(hierarchical_label "LIGHTS_HI"
+		(shape input)
+		(at 68.58 80.01 0)
+		(effects
+			(font

Commit message: Corrected all rececptacle/plug polarity and naming.
Parts:
- GTP: renamed from GTPP; value DTM4 -> DTM4R
- GTP: renamed from GTPR; value DTM4 -> DTM4P
Connections:
- net Earth: now also GTP.4 (Pin_4); no longer GTP.4 (Pin_4)
- net at GTP59.B (SENSE): now also GTP.3 (Pin_3); no longer GTP.3 (Pin_3)
- net at GTP59.O (LOW): now also GTP.2 (Pin_2); no longer GTP.2 (Pin_2)
- net at GTP59.W (POWER): now also GTP.1 (Pin_1); no longer GTP.1 (Pin_1)
- net at GSU25.P252_1 (OAT_POWER): now also GTP.1 (Pin_1); no longer GTP.1 (Pin_1)
- net at GSU25.P252_2 (OAT_HIGH): now also GTP.3 (Pin_3); no longer GTP.3 (Pin_3)
- net at GSU25.P252_3 (OAT_LOW): now also GTP.2 (Pin_2); no longer GTP.2 (Pin_2)
Other:
- moved on the sheet: GTP
