File: electrical/power.kicad_sch (KiCad schematic)
At the start: 67 parts

Commit message: Corrected all rececptacle/plug polarity and naming.
Parts:
- removed ROLR: DTM6, symbol Connector:Conn_01x06_Socket
- added ROL: DTM6R, symbol Connector:Conn_01x06_Pin
- FLP: renamed from FLPP; value DT4 -> DT4R
- FLP: renamed from FLPR; value DT4 -> DT4P
- GMU: renamed from GMUP; value DTM6 -> DTM6R
- GMU: renamed from GMUR; value DTM6 -> DTM6P
- LT: renamed from POTR; value DTM3R -> DTM3P
- LT: renamed from POTP; value DTM3P -> DTM3R
- PIT: renamed from PITR; value DTM6 -> DTM6R
- PIT: renamed from PITP; value DTM6 -> DTM6R
- POS: renamed from POSR; value DTM3 -> DTM3P
- POS: renamed from POSP; value DTM3 -> DTM3R
- PWR: renamed from PWRP; value DTP4 -> DTP4R
- PWR: renamed from PWRR; value DTP4 -> DTP4P
- STB: renamed from STBP; value DT6 -> DT6R
- STB: renamed from STBR; value DT6 -> DT6P
- STK: renamed from STKP; value DTM8 -> DTM8R
- STK: renamed from STKR; value DTM8 -> DTM8P
Connections:
- net 12V_PWR: now also PWR.1 (Pin_1); no longer PWR.1 (Pin_1)
- net CABIN_PWR: now also GMU.5 (Pin_5); no longer GMU.5 (Pin_5)
- net CAMERA_PWR: now also GMU.4 (Pin_4); no longer GMU.4 (Pin_4)
- net FLAPS_1: now also FLP.1 (Pin_1); no longer FLP.1 (Pin_1)
- net FLAPS_2: now also FLP.2 (Pin_2); no longer FLP.2 (Pin_2)
- net FLAPS_DOWN: now also STK.7 (Pin_7); no longer STK.7 (Pin_7)
- net FLAPS_GND: now also POS.3 (Pin_3); no longer POS.3 (Pin_3)
- net FLAPS_POS: now also POS.2 (Pin_2); no longer POS.2 (Pin_2)
- net FLAPS_REF: now also POS.1 (Pin_1); no longer POS.1 (Pin_1)
- net FLAPS_UP: now also STK.6 (Pin_6); no longer STK.6 (Pin_6)
- net FUEL_PWR: now also PWR.3 (Pin_3); no longer PWR.3 (Pin_3)
- net GND: now also FLP.4 (Pin_4), GMU.6 (Pin_6), LT.3 (Pin_3), PIT.6 (Pin_6), PWR.4 (Pin_4), STB.3 (Pin_3), STB.4 (Pin_4), STK.1 (Pin_1); no longer FLP.4 (Pin_4), GMU.6 (Pin_6), LT.3 (Pin_3), PIT.6 (Pin_6), PWR.4 (Pin_4), STB.3 (Pin_3), STB.4 (Pin_4), STK.1 (Pin_1)
- net LEFT_LIGHT_PWR: now also STB.5 (Pin_5); no longer STB.5 (Pin_5)
- net LIGHTS_HI: now also LT.2 (Pin_2); no longer LT.2 (Pin_2)
- net PANEL_PWR: now also LT.1 (Pin_1); no longer LT.1 (Pin_1)
- net PILOT_PTT: now also STK.8 (Pin_8); no longer STK.8 (Pin_8)
- net PITCH_GND: now also PIT.1 (Pin_1); no longer PIT.1 (Pin_1)
- net PITCH_POS: now also PIT.2 (Pin_2); no longer PIT.2 (Pin_2)
- net PITCH_REF: now also PIT.3 (Pin_3); no longer PIT.3 (Pin_3)
- net POSITION_PWR: now also STB.1 (Pin_1); no longer STB.1 (Pin_1)
- net RIGHT_LIGHT_PWR: now also STB.6 (Pin_6); no longer STB.6 (Pin_6)
- net ROLL_GND: now also ROL.1 (Pin_1)
- net ROLL_POS: now also ROL.2 (Pin_2)
- net ROLL_REF: now also ROL.3 (Pin_3)
- net ROLL_TRIM_1: now also ROL.5 (Pin_5)
- net ROLL_TRIM_2: now also ROL.4 (Pin_4)
- net SMOKE_PWR: now also FLP.3 (Pin_3); no longer FLP.3 (Pin_3)
- net STROBE_PWR: now also STB.2 (Pin_2); no longer STB.2 (Pin_2)
- net TRIM_DOWN: now also STK.3 (Pin_3); no longer STK.3 (Pin_3)
- net TRIM_LEFT: now also STK.4 (Pin_4); no longer STK.4 (Pin_4)
- net TRIM_RIGHT: now also STK.5 (Pin_5); no longer STK.5 (Pin_5)
- net TRIM_UP: now also STK.2 (Pin_2); no longer STK.2 (Pin_2)
- net at TRIM_UP_SW.1: now also STK.2 (Pin_2); no longer STK.2 (Pin_2)
- net at CWS_SW.2, FLAPS_DN_SW.2, FLAPS_UP_SW.2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: now also STK.1 (Pin_1); no longer STK.1 (Pin_1)
- net at LEFT_POS.1, RIGHT_POS.1, TAIL_POS.1: now also STB.1 (Pin_1); no longer STB.1 (Pin_1)
- net at BOTTOM_STROBE.R (PWR), TOP_STROBE.R (PWR): now also STB.2 (Pin_2); no longer STB.2 (Pin_2)
- net at BOTTOM_STROBE.B (GROUND), LEFT_LT.2, LEFT_POS.2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: now also STB.3 (Pin_3); no longer STB.3 (Pin_3)
- net at LEFT_LT.1: now also STB.5 (Pin_5); no longer STB.5 (Pin_5)
- net at RIGHT_LT.1: now also STB.6 (Pin_6); no longer STB.6 (Pin_6)
- net at PITCH_POS.O (+5V): now also PIT.1 (Pin_1); no longer PIT.1 (Pin_1)
- net at PITCH_POS.G (SENSE): now also PIT.2 (Pin_2); no longer PIT.2 (Pin_2)
- net at PITCH_POS.B (LOW): now also PIT.3 (Pin_3); no longer PIT.3 (Pin_3)
- net at TRIM_RIGHT_SW.1: now also STK.5 (Pin_5); no longer STK.5 (Pin_5)
- net at CAMERA.1: now also GMU.4 (Pin_4); no longer GMU.4 (Pin_4)
- net at CABIN_LT1.2, CABIN_LT2.2, CAMERA.2: now also GMU.6 (Pin_6); no longer GMU.6 (Pin_6)
- net at FLAPS.1 (+): now also FLP.1 (Pin_1); no longer FLP.1 (Pin_1)
- net at FLAPS.2 (-): now also FLP.2 (Pin_2); no longer FLP.2 (Pin_2)
- net at SMOKE.1 (+): now also FLP.3 (Pin_3); no longer FLP.3 (Pin_3)
- net at SMOKE.2 (-): now also FLP.4 (Pin_4); no longer FLP.4 (Pin_4)
- net at CABIN_LT1.1, CABIN_LT2.1: now also GMU.5 (Pin_5); no longer GMU.5 (Pin_5)
- net at FLAPS_POS.B (LOW): now also POS.3 (Pin_3); no longer POS.3 (Pin_3)
- net at FLAPS_POS.G (SENSE): now also POS.2 (Pin_2); no longer POS.2 (Pin_2)
- net at FLAPS_POS.O (+5V): now also POS.1 (Pin_1); no longer POS.1 (Pin_1)
- net at FLAPS_DN_SW.1: now also STK.7 (Pin_7); no longer STK.7 (Pin_7)
- net at FUEL_PUMP.2 (-), PASSENGER12V.1, PASSENGERUSB.1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: now also PWR.4 (Pin_4); no longer PWR.4 (Pin_4)
- net at PASSENGER12V.2, PASSENGERUSB.2, PILOT12V.2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: now also PWR.1 (Pin_1); no longer PWR.1 (Pin_1)
- net at TRIM_DN_SW.1: now also STK.3 (Pin_3); no longer STK.3 (Pin_3)
- net at LIGHTS_POT.1: now also LT.1 (Pin_1); no longer LT.1 (Pin_1)
- net at LIGHTS_POT.2: now also LT.2 (Pin_2); no longer LT.2 (Pin_2)
- net at LIGHTS_POT.3: now also LT.3 (Pin_3); no longer LT.3 (Pin_3)
- net at FLAPS_UP_SW.1: now also STK.6 (Pin_6); no longer STK.6 (Pin_6)
- net at PILOT_PTT_SW.1: now also STK.8 (Pin_8); no longer STK.8 (Pin_8)
- net at FUEL_PUMP.1 (+): now also PWR.3 (Pin_3); no longer PWR.3 (Pin_3)
- net at TRIM_LEFT_SW.1: now also STK.4 (Pin_4); no longer STK.4 (Pin_4)
Other:
- moved on the sheet: FLP, GMU, LT, PIT, POS, PWR, STB, STK
