File: electrical/lycoming.kicad_sch (KiCad schematic)
At the start: 24 parts

Commit message: Added shielding and wire colors and corrections.
Parts:
- BAT_FUSE: value 80A -> 250A
Changed lines of the file:
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@@
 	(title_block
 		(title "Lycoming")
-		(date "2025-11-03")
-		(rev "1.2.2")
+		(date "2025-11-12")
+		(rev "1.2.5")
 		(company "N78HR")
 	)
@@
 			)
 		)
-		(property "Value" "80A"
+		(property "Value" "250A"
 			(at 64.77 95.2499 0)
 			(effects

Commit message: Removed ground wire to surefly left ignition. Added GPS antenna to GDU.
Connections:
- net Earth: no longer PLD.2 (Pin_2), SFLY_LEFT. (PLEAD)
- new net: PLD.2 (Pin_2), SFLY_LEFT. (PLEAD)
- no-connect marks 8 -> 9
Other:
- note added: "Followed instructions so ground wire coiled up"
- note removed: "Separate ground wires for each SureFly"
Changed lines of the file:
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@@
 	(title_block
 		(title "Lycoming")
-		(date "2025-11-19")
-		(rev "1.2.8")
+		(date "2025-12-20")
+		(rev "1.2.11")
 		(company "N78HR")
 	)
-	(text "Separate ground wires\nfor each SureFly"
+	(text "Followed instructions so\nground wire coiled up"
 		(exclude_from_sim no)
 		(at 104.14 133.858 0)
@@
 	)
 	(junction
-		(at 129.54 139.7)
-		(diameter 0)
-		(color 0 0 0 0)
-	)
-	(junction
 		(at 77.47 77.47)
 		(diameter 0)
@@
 	)
 	(no_connect
+		(at 125.73 139.7)
+	)
+	(no_connect
 		(at 52.07 59.69)
 	)
@@
 	(wire
 		(pts
-			(xy 129.54 139.7) (xy 92.71 139.7)
-		)
-		(stroke
-			(width 0)
-			(type default)
-		)
-	)
-	(wire
-		(pts
 			(xy 130.81 152.4) (xy 132.08 152.4)
 		)
@@
 		)
 		(stroke
+			(width 0)
+			(type default)
+		)
+	)
+	(wire
+		(pts
+			(xy 92.71 139.7) (xy 125.73 139.7)
+		)
+		(stroke

Commit message: adds battery fault
Parts:
- added BAT1S, BAT2S: Conn_01x01_Pin, symbol Connector:Conn_01x01_Pin
- added BAT1S, BAT2S: Conn_01x01_Socket, symbol Connector:Conn_01x01_Socket
Connections:
- new net BAK_BAT_FAULT: BAT1S.1 (Pin_1), BAT2S.1 (Pin_1)
